File: 10_Audio_Facile.kicad_sch (KiCad schematic)
At the start: 18 parts

Commit message: ajout in+
Parts:
- removed ?: 220pF, Capacitor_SMD:C_0603_1608Metric, symbol Device:C
- added J7: Conn_01x01, Chimere_mods:Castellated_conn, symbol Connector_Generic:Conn_01x01
- gave numbers to parts that had none: 17
Connections:
- net GND: now also J2.1 (Pin_1); no longer C7.2, J3.1 (Pin_1)
- net OUT_P: now also J7.1 (Pin_1); no longer J5.1 (Pin_1)
- net SD: now also J3.1 (Pin_1); no longer J2.1 (Pin_1)
- net IN renamed IN-
- new net IN+: C7.2, J5.1 (Pin_1)
